File: BQ27541.brd (EAGLE design)
At the start: 34.8 x 13.2 mm, 33 parts, among them U1 BQ27541_DRZ_12

Commit message: Little modify sense resistor nets
Routing:
- net N$1: track 73.3 -> 93.3 mm, vias 4 -> 18
- net GND: track 45.0 -> 47.9 mm
